File: Hardware/Power-and-Audio/AudioPower/AudioPower.kicad_sch (KiCad schematic)
At the start: 53 parts, among them Q1 PMOS, U1 LM2596T-ADJ, U2 LM2596T-ADJ, U3 NE5532, U4 NE5532, U5 NE5532, U7 LM386

Commit message: Power and Audio Systems Final Version
Parts:
- removed C12: 10u, symbol Device:C_Polarized
- removed C2, C6: 5nF, symbol Device:C
- removed C3, C5: 220uF, symbol Device:C_Polarized
- removed C4: 100uF, symbol Device:C_Polarized
- removed D1, D2: 1N5822, Diode_THT:D_DO-201AD_P15.24mm_Horizontal, symbol Diode:1N5822
- removed L1, L2: 33uH, symbol Device:L
- removed R14, R16: 20k, symbol Device:R
- removed R15: 100k, symbol Device:R
- removed R2, R4: 1k, symbol Device:R
- removed R3: 3.1k, symbol Device:R
- removed R5: 100, symbol Device:R
- removed U1, U2: LM2596T-ADJ, Package_TO_SOT_THT:TO-220-5_P3.4x3.7mm_StaggerOdd_Lead3.8mm_Vertical, symbol Regulator_Switching:LM2596T-ADJ
- removed U5: NE5532, symbol Amplifier_Operational:NE5532
- added C14: 10uF, symbol Device:C_Polarized
- added C2: 0.33uF, symbol Device:C_Polarized
- added R20: 10k, symbol Device:R
- added R32: 2.2M, symbol Device:R
- added U1: L7805, symbol Regulator_Linear:L7805
- added U10, U6: NE5532, symbol Amplifier_Operational:NE5532
- added unit 2 of U3
- added U5: NMA1205SC, Converter_DCDC:Converter_DCDC_Murata_NMAxxxxSC_THT, symbol Regulator_Switching:NMA1205SC
- BT1: value 5V -> 6V
- C1: value 100uF -> 0.1uF
- C11: value 10u -> 10uF
- C19: value 220uF -> 10uF
- C9: value 100u -> 1n
- Q1: value PMOS -> IRFU5305
- R1: value 3.1k -> 10k
- R11: value 20k -> 47k
- R12: value 20k -> 10k
- R13: value 100k -> 10k
- R6: value 20k -> 22k
- R7: value 30k -> 33k
- R8, R9: value 20k -> 100k
Connections:
- net +12V: now also U5.1 (VIN+); no longer C1.1
- net +5V: now also R18.1, R20.1; no longer D5.2 (A), R11.2, R8.2
- net 5V_PIC_SEATS: now also C1.1, U1.3 (OUT); no longer R1.1
- net Combined_audio: now also C13.1, R19.1, U4.1; no longer C13.2, RV2.1
- net GND: now also R1.2, R11.2, R12.2, R13.2, C2.2, R32.2, U1.2 (GND), U5.2 (VIN-), U5.5 (0V); no longer C10.2, R12.1, R9.1
- net at C10.1, R8.1: now also U3.6 (-), U3.7; no longer R18.1, R9.2
- net + Differential Signal: now reaches R13.1, U3.3 (+)
- net + Differential Signal: now also C10.2, R18.2; no longer C11.2
- net at R10.1, U4.3 (+): now also R1.1; no longer R18.2
- net Audio_Diff+: no longer names the net of C11.1
- net Audio_Diff+: now also R9.2, U6.1
- net Audio_Diff_+out renamed + Differential Output
- net Audio_Diff_-out: no longer names the net of R17.2
- net Audio_Diff_-out: now also C14.2
- new net: R11.1, U6.3 (+)
- new net: C13.2, R32.1, RV2.1
- new net: R8.2, R9.1, U6.2 (-)
- new net +24V: C2.1, U1.1 (IN)
- new net +6V: D5.2 (A)
- new net - Differential Output: C14.1, U10.1, U10.2 (-)
- new net - Differential Signal: C11.2, R12.1, R20.2, U10.3 (+)
- new net -5V: U5.4 (VOUT-)
- new net PI_Aux_Output_0_DC_Off: U3.5 (+)
- no-connect marks 0 -> 1
Other:
- note added: "Audio Amplification PI Side"
- note added: "DC Offset 0V max amplitude ~0.5V"
- note added: "DC-DC Converter"
- note added: "Dasiy Chain To The Next Seat"
- note added: "LM2576-ADJ"
- note added: "RN1224"
- note added: "Vin+"
- note added: "Vin-"
- note added: "Vout+"
- note added: "Vout-"
- note removed: "Differential audio pair amplification PI Side"
- moved on the sheet: BT1, C13, C17, C18, C19, C20, C7, C8, C9, D3, D4, D5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
